File: _saved_buckboost.sch (KiCad schematic (older format))
At the start: 24 parts, among them K1 CONN_3, SW1 SPST, U1 TPS63060

Commit message: Schematic Largely Done, many footprints chosen, footprint for Inductor custom made.
Parts:
- C1, C2, C3, C4, C5, C6, C7: footprint (none) -> Capacitors_SMD:C_0805_HandSoldering
- K1: footprint (none) -> Pin_Headers:Pin_Header_Straight_1x03
- R1, R2, R3, R4, R5, R6, R7, R8: footprint (none) -> Resistors_SMD:R_0805_HandSoldering
Changed lines of the file:
@@
 LIBS:valves
 LIBS:tps63060
+LIBS:buckboost-cache
 EELAYER 25 0
 EELAYER END
@@
 F 0 "U1" H 4950 5000 60  0000 C CNN
 F 1 "TPS63060" H 4950 4200 60  0000 C CNN
-F 2 "" H 4950 4150 60  0000 C CNN
+F 2 "" H 4950 4150 60  0001 C CNN
 F 3 "" H 4950 4150 60  0000 C CNN
 	1    4950 4150
@@
 F 0 "C2" H 3550 3800 40  0000 L CNN
 F 1 "0.1 uF" H 3556 3615 40  0000 L CNN
-F 2 "" H 3588 3550 30  0000 C CNN
+F 2 "Capacitors_SMD:C_0805_HandSoldering" H 3588 3550 30  0001 C CNN
 F 3 "" H 3550 3700 60  0000 C CNN
 	1    3550 3700
@@
 F 0 "L1" V 4900 3100 40  0000 C CNN
 F 1 "1 uH" V 5050 3100 40  0000 C CNN
-F 2 "" H 4950 3100 60  0000 C CNN
+F 2 "" H 4950 3100 60  0001 C CNN
 F 3 "" H 4950 3100 60  0000 C CNN
 	1    4950 3100
@@
 F 0 "C3" H 4150 4400 40  0000 L CNN
 F 1 "0.1 uF" H 4156 4215 40  0000 L CNN
-F 2 "" H 4188 4150 30  0000 C CNN
+F 2 "Capacitors_SMD:C_0805_HandSoldering" H 4188 4150 30  0001 C CNN
 F 3 "" H 4150 4300 60  0000 C CNN
 	1    4150 4300
@@
 F 0 "R4" V 5930 3600 40  0000 C CNN
 F 1 "1M R" V 5857 3601 40  0000 C CNN
-F 2 "" V 5780 3600 30  0000 C CNN
+F 2 "Resistors_SMD:R_0805_HandSoldering" V 5780 3600 30  0001 C CNN
 F 3 "" H 5850 3600 30  0000 C CNN
 	1    5850 3600
@@
 F 0 "C4" H 6350 4050 40  0000 L CNN
 F 1 "10 pF" H 6356 3865 40  0000 L CNN
-F 2 "" H 6388 3800 30  0000 C CNN
+F 2 "Capacitors_SMD:C_0805_HandSoldering" H 6388 3800 30  0001 C CNN
 F 3 "" H 6350 3950 60  0000 C CNN
 	1    6350 3950
@@
 F 0 "R6" V 7030 3950 40  0000 C CNN
 F 1 "1M R" V 6957 3951 40  0000 C CNN
-F 2 "" V 6880 3950 30  0000 C CNN
+F 2 "Resistors_SMD:R_0805_HandSoldering" V 6880 3950 30  0001 C CNN
 F 3 "" H 6950 3950 30  0000 C CNN
 	1    6950 3950
@@
 F 0 "C5" H 8050 3800 40  0000 L CNN
 F 1 "22uF" H 8056 3615 40  0000 L CNN
-F 2 "" H 8088 3550 30  0000 C CNN
+F 2 "Capacitors_SMD:C_0805_HandSoldering" H 8088 3550 30  0001 C CNN
 F 3 "" H 8050 3700 60  0000 C CNN
 	1    8050 3700
@@
 F 0 "C1" H 3200 3800 40  0000 L CNN
 F 1 "10 uF" H 3206 3615 40  0000 L CNN
-F 2 "" H 3238 3550 30  0000 C CNN
+F 2 "Capacitors_SMD:C_0805_HandSoldering" H 3238 3550 30  0001 C CNN
 F 3 "" H 3200 3700 60  0000 C CNN
 	1    3200 3700
@@
 F 0 "C6" H 8300 3800 40  0000 L CNN
 F 1 "22uF" H 8306 3615 40  0000 L CNN
-F 2 "" H 8338 3550 30  0000 C CNN
+F 2 "Capacitors_SMD:C_0805_HandSoldering" H 8338 3550 30  0001 C CNN
 F 3 "" H 8300 3700 60  0000 C CNN
 	1    8300 3700
@@
 F 0 "C7" H 8550 3800 40  0000 L CNN
 F 1 "22uF" H 8556 3615 40  0000 L CNN
-F 2 "" H 8588 3550 30  0000 C CNN
+F 2 "Capacitors_SMD:C_0805_HandSoldering" H 8588 3550 30  0001 C CNN
 F 3 "" H 8550 3700 60  0000 C CNN
 	1    8550 3700
@@
 F 0 "SW1" H 1200 3600 70  0000 C CNN
 F 1 "SPST" H 1200 3400 70  0000 C CNN
-F 2 "" H 1200 3500 60  0000 C CNN
+F 2 "" H 1200 3500 60  0001 C CNN
 F 3 "" H 1200 3500 60  0000 C CNN
 	1    1200 3500
@@
 F 0 "D1" H 700 3100 40  0000 C CNN
 F 1 "DIODESCH" H 700 2900 40  0000 C CNN
-F 2 "" H 700 3000 60  0000 C CNN
+F 2 "" H 700 3000 60  0001 C CNN
 F 3 "" H 700 3000 60  0000 C CNN
 	1    700  3000
@@
 F 0 "R5" V 6530 3100 40  0000 C CNN
 F 1 "22k R" V 6457 3101 40  0000 C CNN
-F 2 "" V 6380 3100 30  0000 C CNN
+F 2 "Resistors_SMD:R_0805_HandSoldering" V 6380 3100 30  0001 C CNN
 F 3 "" H 6450 3100 30  0000 C CNN
 	1    6450 3100
@@
 F 0 "D3" H 6850 2950 50  0000 C CNN
 F 1 "LED" H 6850 2750 50  0000 C CNN
-F 2 "" H 6850 2850 60  0000 C CNN
+F 2 "" H 6850 2850 60  0001 C CNN
 F 3 "" H 6850 2850 60  0000 C CNN
 	1    6850 2850
@@
 F 0 "R3" V 3030 3750 40  0000 C CNN
 F 1 "22k R" V 2957 3751 40  0000 C CNN
-F 2 "" V 2880 3750 30  0000 C CNN
+F 2 "Resistors_SMD:R_0805_HandSoldering" V 2880 3750 30  0001 C CNN
 F 3 "" H 2950 3750 30  0000 C CNN
 	1    2950 3750
@@
 F 0 "D2" H 2950 4400 50  0000 C CNN
 F 1 "LED" H 2950 4200 50  0000 C CNN
-F 2 "" H 2950 4300 60  0000 C CNN
+F 2 "" H 2950 4300 60  0001 C CNN
 F 3 "" H 2950 4300 60  0000 C CNN
 	1    2950 4300
@@
 F 0 "K1" V 1800 1000 50  0000 C CNN
 F 1 "CONN_3" V 1900 1000 40  0000 C CNN
-F 2 "" H 1850 1000 60  0000 C CNN
+F 2 "Pin_Headers:Pin_Header_Straight_1x03" H 1850 1000 60  0001 C CNN
 F 3 "" H 1850 1000 60  0000 C CNN
 	1    1850 1000
@@
 F 0 "R2" V 1580 1450 40  0000 C CNN
 F 1 "111k R" V 1507 1451 40  0000 C CNN
-F 2 "" V 1430 1450 30  0000 C CNN
+F 2 "Resistors_SMD:R_0805_HandSoldering" V 1430 1450 30  0001 C CNN
 F 3 "" H 1500 1450 30  0000 C CNN
 	1    1500 1450
@@
 F 0 "R1" V 830 1450 40  0000 C CNN
 F 1 "179k R" V 757 1451 40  0000 C CNN
-F 2 "" V 680 1450 30  0000 C CNN
+F 2 "Resistors_SMD:R_0805_HandSoldering" V 680 1450 30  0001 C CNN
 F 3 "" H 750 1450 30  0000 C CNN
 	1    750  1450
@@
 F 0 "FB1" H 2150 3600 50  0000 C CNN
 F 1 "1K @ 100 MHz" H 2150 3450 50  0000 C CNN
-F 2 "" H 2150 3500 60  0000 C CNN
+F 2 "" H 2150 3500 60  0001 C CNN
 F 3 "" H 2150 3500 60  0000 C CNN
 	1    2150 3500
@@
 F 0 "FB2" H 7600 3600 50  0000 C CNN
 F 1 "1K @ 100 MHz" H 7600 3450 50  0000 C CNN
-F 2 "" H 7600 3500 60  0000 C CNN
+F 2 "" H 7600 3500 60  0001 C CNN
 F 3 "" H 7600 3500 60  0000 C CNN
 	1    7600 3500
@@
 F 0 "R8" V 8980 3500 40  0000 C CNN
 F 1 "0.01" V 8907 3501 40  0000 C CNN
-F 2 "" V 8830 3500 30  0000 C CNN
+F 2 "Resistors_SMD:R_0805_HandSoldering" V 8830 3500 30  0001 C CNN
 F 3 "" H 8900 3500 30  0000 C CNN
 	1    8900 3500
@@
 F 0 "R7" V 4180 3500 40  0000 C CNN
 F 1 "0.01" V 4107 3501 40  0000 C CNN
-F 2 "" V 4030 3500 30  0000 C CNN
+F 2 "Resistors_SMD:R_0805_HandSoldering" V 4030 3500 30  0001 C CNN
 F 3 "" H 4100 3500 30  0000 C CNN
 	1    4100 3500
